File: qrotx-singleband-transmitter/qrotx-singleband-transmitter_RF.kicad_sch (KiCad schematic)
At the start: 61 parts, among them J3 Conn_Coaxial, J4 Conn_Coaxial, K1 G2RL-1, K2 G2RL-1, Q1 IPB085N15NM6, Q2 IPB085N15NM6, Q3 GAN080-650EBE, Q4 GAN080-650EBE, Q5 BSS138, U6 UCC27884DR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

Commit message: Update text blocks in drawings
Other:
- note added: "only place on of the parallel resonators"
Changed lines of the file:
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@@
 	(title_block
 		(title "qrotx Single Band (40m) Transmitter")
-		(date "2026-02-15")
+		(date "2026-04-06")
 		(rev "0")
 		(company "Christian Riesch K2CRI")
 		(comment 1 "Copyright (c) 2024-2026 Christian Riesch, christian@riesch.at")
 		(comment 2 "Licensed under CERN-OHL-S v2 or any later version, https://ohwr.org/cern_ohl_s_v2.txt")
-		(comment 3 "https://www.qrotx.org")
+		(comment 3 "https://qrotx.org")
 	)
 	(text "Balun\n"
@@
 			)
 		)
+	)
+	(text "only place on of the parallel resonators"
+		(exclude_from_sim no)
+		(at 260.35 133.35 0)
+		(effects
+			(font
+				(size 1.27 1.27)
+			)
+		)
